Commit message: work in progress

File: ik_teleop/robot/assets/allegro_hand_right.urdf (robot description, URDF)
Before this commit: robot allegro_hand_right, 21 links, 20 joints
Joints:
- joint joint_12.0: limit lower=0.263 upper=1.396 effort=0 velocity=0 -> lower=0.225 upper=1.555 effort=0 velocity=0
- joint joint_13.0: limit lower=-0.105 upper=2 effort=0 velocity=7 -> lower=-0.368 upper=1.152 effort=0 velocity=0
- joint joint_14.0: limit lower=-0.189 upper=1.644 effort=0 velocity=0 -> lower=-0.281 upper=1.719 effort=0 velocity=0
- joint joint_15.0: limit lower=-0.162 upper=1.719 effort=0 velocity=0 -> lower=-0.262 upper=1.799 effort=0 velocity=0
